File: pcb/RGBClock/Displayboard.sch (EAGLE design)
At the start: 0 parts

Commit message: Mainboard + displayboard
Parts:
- added C4: 2.2uF, AVX_By_element14_Batch_1:08053C225KAT2A
- added CON1: (no value), con-harting:CON20
- added D1, D2: SMA6F, MyComponents:SMA6F
- added D10: HSMS-2800-TR1G, diode:BAS70
- added IC1: MCP23017SO, microchip:MCP23017SO
- added JP1: (no value), jumper:JP1E
- added L1: 68uH, WE-PD4:WE-PD4-74456168_L
- added R5, R7: 3300, rcl:R-EU_0204/7
- added R8: 0.3R, resistor:R-EU_R0603
- added U$1: TPA0172-HTSSOP24, MyComponents:TPA0172-HTSSOP24
- added U1, U4: P82B96DR, Texas:P82B96DR
- added U2: TPS71533DCKR, Texas:TPS71533DCKR
- added U5: PCA9685PW, NXP_By_element14_Batch_1:PCA9685PW
- added U6: ZXLD1362ET5TA, ZEtex:ZXLD1362ET5TA
- added X1: 5566-4, con-molex:5566-4
- added X2: 5566-2, con-molex:5566-2
Connections:
- new net +5V: R5.2, R7.2, U4.VCC, U5.VDD
- new net GND: C4.C1, D1.AN, D2.AN, U4.GND, U5.A0, U5.A1, U5.A2, U5.A3, U5.A4, U5.A5, U5.EXTCLK, U5.VSS, U5.~OE, U6.GND
- new net N$1: JP1.1, R8.1, U6.ISENSE
- new net N$10: D10.A, L1.1, U6.LX
- new net N$12: R5.1, U4.SY, U5.SCL
- new net N$17: D1.KAT, U4.RX, U4.TX, X1-2.S
- new net N$22: D2.KAT, U4.RY, U4.TY, X1-1.S
- new net N$3: R7.1, U4.SX, U5.SDA
- new net N$6: JP1.2, L1.2
- new net N$8: U5.LED0, U6.ADJ
- new net VCC: C4.C2, D10.C, R8.2, U6.VIN
