File: pcb/RGBClock/Displayboard.sch (EAGLE design)
At the start: 66 parts, among them IC1 MCP23017SO, U1 LP3878MR-ADJ, U2 P82B96DR, U3 P82B96DR, U4 PCA9685PW, U5 TPS71533DCKR, U6 ZXLD1362ET5TA, U7 74HCT1G14GW, U8 74HCT1G86GW, X1 43045-0400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

Commit message: Mainboard routable !
Parts:
- renumbered IC1 to U10, U$1 to U9
