File: pcb/RGBClock/Leddriverboard.sch (EAGLE design)
At the start: 0 parts

Commit message: Mainboard, Displayboard, Leddriverboard
Parts:
- added C1: 4u7, rcl:C-EUC1206
- added C2: 10n, rcl:C-EUC1608
- added C3: 680p, rcl:C-EUC1608
- added C4: 10u, rcl:C-EUC2012
- added C5, C6, C7: 2.2uF, AVX_By_element14_Batch_1:08053C225KAT2A
- added D1: MUR480ERLG, diode:MUR150RL
- added D2, D3: SMA6F, MyComponents:SMA6F
- added D4, D5, D6: VS-30BQ100PBF, MyComponents:VS-30BQ100PBF
- added L1, L2, L3: 68uH, WE-PD4:WE-PD4-74456168_L
- added R1: 4.02k, resistor:R-EU_R0603
- added R10, R7: 3300, rcl:R-EU_0204/7
- added R11, R12, R13: 0.3R, resistor:R-EU_R0603
- added R2: 1k, resistor:R-EU_R0603
- added R3: A2-1, resistor:R-EU_R0402
- added R4: A2-0, resistor:R-EU_R0402
- added R5: A1-1, resistor:R-EU_R0402
- added R6: A1-0, resistor:R-EU_R0402
- added R8: A0-1, resistor:R-EU_R0402
- added R9: A0-0, resistor:R-EU_R0402
- added U1: LP3878MR-ADJ, Texas:LP3878MR-ADJ
- added U2: P82B96DR, Texas:P82B96DR
- added U3: PCA9685PW, NXP_By_element14_Batch_1:PCA9685PW
- added U4, U5, U6: ZXLD1362ET5TA, ZEtex:ZXLD1362ET5TA
- added X1: 5566-4, con-molex:5566-4
- added X2: (no value), con-molex-micro-fit-3_0:HEADER_POS6_43045-0600
Connections:
- new net +5V: C3.1, C4.1, R1.1, R10.2, R3.2, R5.2, R7.2, R8.2, U1.OUT, U2.VCC, U3.VDD
- new net GND: C1.2, C2.2, C4.2, C5.C1, C6.C1, C7.C1, D2.AN, D3.AN, R2.2, R4.1, R6.1, R9.1, U1.GND, U1.GND_2, U2.GND, U3.A3, U3.A4, U3.A5, U3.EXTCLK, U3.VSS, U3.~OE, U4.GND, U5.GND, U6.GND, X1-3.S
- new net N$1: R11.1, U4.ISENSE, X2.1
- new net N$10: D4.A, L1.1, U4.LX
- new net N$15: U3.LED2, U6.ADJ
- new net N$16: R13.1, U6.ISENSE, X2.5
- new net N$18: L3.2, X2.6
- new net N$19: D6.A, L3.1, U6.LX
- new net N$2: U3.LED1, U5.ADJ
- new net N$22: D2.KAT, U2.RY, U2.TY, X1-1.S
- new net N$24: C3.2, R1.2, R2.1, U1.ADJ
- new net N$25: D1.A, X1-4.S
- new net N$26: C2.1, U1.BYPASS
- new net N$4: R12.1, U5.ISENSE, X2.3
- new net N$41: R8.1, R9.2, U3.A0
- new net N$42: R5.1, R6.2, U3.A1
- new net N$43: R3.1, R4.2, U3.A2
- new net N$5: L2.2, X2.4
- new net N$6: L1.2, X2.2
- new net N$7: D3.KAT, U2.RX, U2.TX, X1-2.S
- new net N$8: U3.LED0, U4.ADJ
- new net N$9: D5.A, L2.1, U5.LX
- new net SCL: R7.1, U2.SY, U3.SCL
- new net SDA: R10.1, U2.SX, U3.SDA
- new net VCC: C1.1, C5.C2, C6.C2, C7.C2, D1.C, D4.C, D5.C, D6.C, R11.2, R12.2, R13.2, U1.IN, U1.~SD, U4.VIN, U5.VIN, U6.VIN
