File: pcb/RGBClock/Leddriverboard.sch (EAGLE design)
At the start: 37 parts, among them U1 LP3878MR-ADJ, U2 P82B96DR, U3 PCA9685PW, U4 ZXLD1362ET5TA, U5 ZXLD1362ET5TA, U6 ZXLD1362ET5TA, X1 43045-0400, X2 43045-0600

Commit message: Main and Display updated
Parts:
- C1: device rcl:C-EUC1206 -> rcl:C-EUC0805
- C2, C3: device rcl:C-EUC1608 -> rcl:C-EUC0805
- C4: device rcl:C-EUC2012 -> rcl:C-EUC0805
Changed lines of the file:
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@@
 <part name="P+3" library="supply1" deviceset="+5V" device=""/>
 <part name="GND16" library="supply1" deviceset="GND" device=""/>
-<part name="C1" library="rcl" deviceset="C-EU" device="C1206" value="4u7"/>
-<part name="C2" library="rcl" deviceset="C-EU" device="C1608" value="10n"/>
-<part name="C3" library="rcl" deviceset="C-EU" device="C1608" value="680p"/>
+<part name="C1" library="rcl" deviceset="C-EU" device="C0805" value="4u7"/>
+<part name="C2" library="rcl" deviceset="C-EU" device="C0805" value="10n"/>
+<part name="C3" library="rcl" deviceset="C-EU" device="C0805" value="680p"/>
 <part name="R1" library="resistor" deviceset="R-EU_" device="R0603" value="4.02k"/>
 <part name="R2" library="resistor" deviceset="R-EU_" device="R0603" value="1k"/>
 <part name="GND20" library="supply1" deviceset="GND" device=""/>
-<part name="C4" library="rcl" deviceset="C-EU" device="C2012" value="10u"/>
+<part name="C4" library="rcl" deviceset="C-EU" device="C0805" value="10u"/>
 <part name="GND21" library="supply1" deviceset="GND" device=""/>
 <part name="GND22" library="supply1" deviceset="GND" device=""/>
