File: pcb/RGBClock/Leddriverboard.brd (EAGLE design)
At the start: 70 x 47.5 mm, 37 parts, among them U1 LP3878MR-ADJ, U2 P82B96DR, U3 PCA9685PW, U4 ZXLD1362ET5TA, U5 ZXLD1362ET5TA, U6 ZXLD1362ET5TA, X1 43045-0400, X2 43045-0600

Commit message: Main and Display updated
Parts:
- C1: device rcl:C1206 -> rcl:C0805
- C2, C3: device rcl:C1608 -> rcl:C0805
- C4: device rcl:C2012 -> rcl:C0805
Routing:
- net GND: track 220.2 -> 0.00 mm, vias 2 -> 0
- net VCC: track 155.7 -> 0.00 mm
- net +5V: track 69.8 -> 0.00 mm, vias 1 -> 0
- net N$15: track 46.6 -> 0.00 mm
- net N$8: track 45.1 -> 0.00 mm, vias 2 -> 0
- net N$22: track 41.8 -> 0.00 mm
- net SCL: track 35.3 -> 0.00 mm
- net SDA: track 32.5 -> 0.00 mm
- net N$16: track 30.9 -> 0.00 mm
- net N$2: track 27.2 -> 0.00 mm
- net N$4: track 25.0 -> 0.00 mm, vias 1 -> 0
- net N$19: track 22.6 -> 0.00 mm
- net N$9: track 18.8 -> 0.00 mm
- net N$5: track 18.7 -> 0.00 mm
- net N$41: track 16.3 -> 0.00 mm
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- removed copper zone on layer 1, net GND
- removed copper zone on layer 16, net GND

Commit message: Ready
Parts:
- moved R11 1.80 mm to (56.7, 34.7)
- moved U4 1.58 mm to (56.7, 31.0)
- moved C5 1.12 mm to (53.1, 31.0)
Routing:
- net GND: track 0.00 -> 170.3 mm
- net VCC: track 0.00 -> 162.3 mm, vias 0 -> 2
- net +5V: track 0.00 -> 70.5 mm, vias 0 -> 1
- net N$15: track 0.00 -> 46.6 mm
- net N$8: track 0.00 -> 45.2 mm, vias 0 -> 2
- net N$22: track 0.00 -> 41.7 mm
- net SCL: track 0.00 -> 38.5 mm
- net SDA: track 0.00 -> 32.6 mm
- net N$16: track 0.00 -> 30.9 mm
- net N$2: track 0.00 -> 26.9 mm
- net N$4: track 0.00 -> 25.1 mm, vias 0 -> 1
- net N$19: track 0.00 -> 22.6 mm
- net N$5: track 0.00 -> 18.7 mm
- net N$9: track 0.00 -> 18.1 mm
- net N$1: track 0.00 -> 16.6 mm
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- added copper zone on layer 1, net GND
- added copper zone on layer 16, net GND
