File: pcb/RGBClock/Mainboard.sch (EAGLE design)
At the start: 106 parts, among them IC1 MCP23017SO, IC2 LT1763CS8-1.5, K1 G6K-2F, K2 G6K-2F, K3 G6K-2F, K4 G6K-2F, Q1 32.768KHz, U1 MAX6369KA+T, U10 NX3L1G384GW, U11 NX3L1G384GW, U13 DRV612PW, U14 2N7002-7-F, U15 2N7002-7-F, U16 2N7002-7-F, U17 2N7002-7-F, U2 TXS0102DCUR, U3 P82B96DR, U4 LM2675M-5.0, U5 DS1338Z-33+, U7 TPS71533DCKR, U8 NX3L1G384GW, U9 NX3L1G384GW, X2 43045-0400, X3 CON-LUMBERG_1503_09, X4 CON-LUMBERG_1503_09, X5 43045-0800, X6 ST-SMB-H

Commit message: dab routed manually
Connections:
- removed net +24V: C11.1, C12.1, C13.1, C22.1, C28.2, C29.2, U$2.VA, U$2.VCORE, U$2.VMEM
- net +1.8V: now also C11.1, C12.1, C13.1, C22.1, C28.2, C29.2, U$2.VA, U$2.VCORE, U$2.VMEM
Changed lines of the file:
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@@
 <setting verticaltext="up"/>
 </settings>
-<grid distance="1" unitdist="mm" unit="mm" style="lines" multiple="1" display="no" altdistance="0.01" altunitdist="inch" altunit="inch"/>
+<grid distance="0.1" unitdist="inch" unit="inch" style="lines" multiple="1" display="no" altdistance="0.01" altunitdist="inch" altunit="inch"/>
 <layers>
 <layer number="1" name="Top" color="4" fill="1" visible="no" active="no"/>
@@
 </variantdefs>
 <classes>
-<class number="0" name="default" width="0.2032" drill="0">
-<clearance class="0" value="0.1524"/>
+<class number="0" name="default" width="0.254" drill="0">
+<clearance class="0" value="0.254"/>
 </class>
 <class number="1" name="Normal Bcc" width="0.254" drill="0">
@@
 <class number="3" name="LED Current" width="0.381" drill="0">
 <clearance class="3" value="0.254"/>
+</class>
+<class number="4" name="DABChip" width="0.1524" drill="0">
+<clearance class="4" value="0.1524"/>
 </class>
 </classes>
@@
 <part name="GND51" library="Mainboard" deviceset="SUPPLY1_GND" device="" value="GND"/>
 <part name="GND52" library="Mainboard" deviceset="SUPPLY1_GND" device="" value="GND"/>
-<part name="P+25" library="Mainboard" deviceset="SUPPLY1_+24V" device="" value="+1.8V"/>
 <part name="P+26" library="Mainboard" deviceset="SUPPLY1_+24V" device="" value="+1.8V"/>
 <part name="+3V10" library="Mainboard" deviceset="SUPPLY1_+3V3" device="" value="+3V3"/>
@@
 <part name="JP2" library="Mainboard" deviceset="JUMPER_JP1E" device=""/>
 <part name="+3V19" library="Mainboard" deviceset="SUPPLY1_+3V3" device="" value="+3V3"/>
+<part name="P+6" library="Mainboard" deviceset="SUPPLY1_+24V" device="" value="+1.8V"/>
 </parts>
 <sheets>
@@
 <attribute name="VALUE" x="107.95" y="-21.59" size="1.778" layer="96"/>
 </instance>
-<instance part="P+25" gate="1" x="111.76" y="113.03" smashed="yes">
-<attribute name="VALUE" x="109.22" y="109.22" size="1.778" layer="96" rot="R90"/>
-</instance>
 <instance part="P+26" gate="1" x="149.86" y="83.82" smashed="yes" rot="R270">
 <attribute name="VALUE" x="149.86" y="86.36" size="1.778" layer="96"/>
@@
 <instance part="+3V19" gate="G$1" x="261.62" y="121.92" smashed="yes">
 <attribute name="VALUE" x="264.16" y="124.46" size="1.778" layer="96" rot="R180"/>
+</instance>
+<instance part="P+6" gate="1" x="111.76" y="114.3" smashed="yes">
+<attribute name="VALUE" x="119.38" y="119.38" size="1.778" layer="96" rot="R180"/>
 </instance>
 </instances>
@@
 </busses>
 <nets>
-<net name="GND" class="0">
+<net name="GND" class="4">
 <segment>
 <pinref part="U2" gate="A" pin="GND"/>
@@
 </segment>
 </net>
-<net name="+3V3" class="1">
+<net name="+3V3" class="4">
 <segment>
 <pinref part="+3V2" gate="G$1" pin="+3V3"/>
@@
 </segment>
 </net>
-<net name="N$27" class="0">
+<net name="N$27" class="4">
 <segment>
 <pinref part="U8" gate="A" pin="Y"/>
@@
 </segment>
 </net>
-<net name="N$35" class="0">
+<net name="N$35" class="4">
 <segment>
 <wire x1="63.5" y1="33.02" x2="233.68" y2="33.02" width="0.1524" layer="91"/>
@@
 </segment>
 </net>
-<net name="SDA" class="0">
+<net name="SDA" class="4">
 <segment>
 <pinref part="U3" gate="A" pin="SX"/>
@@
 </segment>
 </net>
-<net name="SCL" class="0">
+<net name="SCL" class="4">
 <segment>
 <pinref part="U2" gate="A" pin="B2"/>
@@
 <wire x1="241.3" y1="152.4" x2="241.3" y2="149.86" width="0.1524" layer="91"/>
 <junction x="241.3" y="149.86"/>
-</segment>
-</net>
-<net name="N$2" class="0">
+<label x="248.92" y="149.86" size="1.778" layer="95"/>
+</segment>
+<segment>
+<pinref part="P+24" gate="1" pin="+24V"/>
+<pinref part="U$2" gate="G$1" pin="VA"/>
+<wire x1="43.18" y1="58.42" x2="66.04" y2="58.42" width="0.1524" layer="91"/>
+<pinref part="C22" gate="G$1" pin="1"/>
+<pinref part="C12" gate="G$1" pin="1"/>
+<wire x1="66.04" y1="38.1" x2="66.04" y2="43.18" width="0.1524" layer="91"/>
+<wire x1="66.04" y1="43.18" x2="66.04" y2="58.42" width="0.1524" layer="91"/>
+<junction x="66.04" y="43.18"/>
+<junction x="66.04" y="58.42"/>
+</segment>
+<segment>
+<pinref part="U$2" gate="G$1" pin="VMEM"/>
+<pinref part="C11" gate="G$1" pin="1"/>
+<wire x1="129.54" y1="83.82" x2="140.97" y2="83.82" width="0.1524" layer="91"/>
+<pinref part="C13" gate="G$1" pin="1"/>
+<wire x1="140.97" y1="83.82" x2="146.05" y2="83.82" width="0.1524" layer="91"/>
+<junction x="140.97" y="83.82"/>
+<pinref part="P+26" gate="1" pin="+24V"/>
+<wire x1="147.32" y1="83.82" x2="146.05" y2="83.82" width="0.1524" layer="91"/>
+<junction x="146.05" y="83.82"/>
+</segment>
+<segment>
+<pinref part="U$2" gate="G$1" pin="VCORE"/>
+<wire x1="111.76" y1="99.06" x2="111.76" y2="101.6" width="0.1524" layer="91"/>
+<pinref part="C28" gate="G$1" pin="2"/>
+<wire x1="111.76" y1="101.6" x2="111.76" y2="106.68" width="0.1524" layer="91"/>
+<wire x1="111.76" y1="106.68" x2="111.76" y2="107.95" width="0.1524" layer="91"/>
+<wire x1="116.84" y1="107.95" x2="111.76" y2="107.95" width="0.1524" layer="91"/>
+<pinref part="C29" gate="G$1" pin="2"/>
+<wire x1="116.84" y1="101.6" x2="111.76" y2="101.6" width="0.1524" layer="91"/>
+<junction x="111.76" y="101.6"/>
+<pinref part="P+6" gate="1" pin="+24V"/>
+<wire x1="111.76" y1="111.76" x2="111.76" y2="107.95" width="0.1524" layer="91"/>
+</segment>
+</net>
+<net name="N$2" class="4">
 <segment>
 <pinref part="U$2" gate="G$1" pin="XTALI"/>
@@
 </segment>
 </net>
-<net name="N$26" class="0">
+<net name="N$26" class="4">
 <segment>
 <pinref part="U$2" gate="G$1" pin="XTALO"/>
@@
 </segment>
 </net>
-<net name="N$34" class="0">
+<net name="N$34" class="4">
 <segment>
 <pinref part="U9" gate="A" pin="Y"/>
@@
 </segment>
 </net>
-<net name="+24V" class="0">
-<segment>
-<pinref part="P+24" gate="1" pin="+24V"/>
-<pinref part="U$2" gate="G$1" pin="VA"/>
-<wire x1="43.18" y1="58.42" x2="66.04" y2="58.42" width="0.1524" layer="91"/>
-<pinref part="C22" gate="G$1" pin="1"/>
-<pinref part="C12" gate="G$1" pin="1"/>
-<wire x1="66.04" y1="38.1" x2="66.04" y2="43.18" width="0.1524" layer="91"/>
-<wire x1="66.04" y1="43.18" x2="66.04" y2="58.42" width="0.1524" layer="91"/>
-<junction x="66.04" y="43.18"/>
-<junction x="66.04" y="58.42"/>
-</segment>
-<segment>
-<pinref part="U$2" gate="G$1" pin="VMEM"/>
-<pinref part="C11" gate="G$1" pin="1"/>
-<wire x1="129.54" y1="83.82" x2="140.97" y2="83.82" width="0.1524" layer="91"/>
-<pinref part="C13" gate="G$1" pin="1"/>
-<wire x1="140.97" y1="83.82" x2="146.05" y2="83.82" width="0.1524" layer="91"/>
-<junction x="140.97" y="83.82"/>
-<pinref part="P+26" gate="1" pin="+24V"/>
-<wire x1="147.32" y1="83.82" x2="146.05" y2="83.82" width="0.1524" layer="91"/>
-<junction x="146.05" y="83.82"/>
-</segment>
-<segment>
-<pinref part="U$2" gate="G$1" pin="VCORE"/>
-<pinref part="P+25" gate="1" pin="+24V"/>
-<wire x1="111.76" y1="99.06" x2="111.76" y2="101.6" width="0.1524" layer="91"/>
-<pinref part="C28" gate="G$1" pin="2"/>
-<wire x1="111.76" y1="101.6" x2="111.76" y2="107.95" width="0.1524" layer="91"/>
-<wire x1="111.76" y1="107.95" x2="111.76" y2="110.49" width="0.1524" layer="91"/>
-<wire x1="116.84" y1="107.95" x2="111.76" y2="107.95" width="0.1524" layer="91"/>
-<junction x="111.76" y="107.95"/>
-<pinref part="C29" gate="G$1" pin="2"/>
-<wire x1="116.84" y1="101.6" x2="111.76" y2="101.6" width="0.1524" layer="91"/>
-<junction x="111.76" y="101.6"/>
-</segment>
-</net>
-<net name="N$68" class="0">
+<net name="N$68" class="4">
 <segment>
 <pinref part="U$2" gate="G$1" pin="ABYP"/>
@@
 </segment>
 </net>
-<net name="N$69" class="0">
+<net name="N$69" class="4">
 <segment>
 <pinref part="C23" gate="G$1" pin="2"/>
@@
 </segment>
 </net>
-<net name="N$70" class="0">
+<net name="N$70" class="4">
 <segment>
 <pinref part="U$2" gate="G$1" pin="DBYP"/>
@@
 </segment>
 </net>
-<net name="N$14" class="0">
+<net name="N$14" class="4">
 <segment>
 <pinref part="R20" gate="G$1" pin="1"/>
@@
 </segment>
 </net>
-<net name="N$65" class="0">
+<net name="N$65" class="4">
 <segment>
 <pinref part="R22" gate="G$1" pin="1"/>

Commit message: juiste positie
Parts:
- removed R20: A0-1, Mainboard:RESISTOR_R-EU_R0402:1
- removed R21: A0-0, Mainboard:RESISTOR_R-EU_R0402:1
- removed R22: A1-1, Mainboard:RESISTOR_R-EU_R0402:1
- removed R24: A1-0, Mainboard:RESISTOR_R-EU_R0402:1
- removed U$2: SI4684-A10, Mainboard:MAINBOARD_SI4684-A10-GMQF
- added U$6: SI4684-MYSMD, Mainboard:SI4684-MYSMD
Connections:
- removed net N$14: R20.1, R21.2, U$2.MISO
- removed net N$65: R22.1, R24.2, U$2.SSB
- new net N$62: U$6.SMODE
- net +1.8V: now also U$6.VA, U$6.VCORE, U$6.VMEM; no longer U$2.VA, U$2.VCORE, U$2.VMEM
- net +3V3: now also U$6.VIO; no longer R20.2, R22.2, U$2.SMODE, U$2.VIO
- net GND: now also U$6.GNDD1, U$6.GNDD2, U$6.GNDD3, U$6.GNDD4, U$6.MISO, U$6.RFREF1, U$6.RFREF2, U$6.RFREF3, U$6.RFREF4, U$6.SSB; no longer R21.1, R24.1, U$2.GNDD1, U$2.GNDD2, U$2.GNDD3, U$2.GNDD4, U$2.RFREF1, U$2.RFREF2, U$2.RFREF3, U$2.RFREF4
- net N$2: now also U$6.XTALI; no longer U$2.XTALI
- net N$26: now also U$6.XTALO; no longer U$2.XTALO
- net N$27: now also U$6.LOUT; no longer U$2.LOUT
- net N$32: now also U$6.VHFSW; no longer U$2.VHFSW
- net N$34: now also U$6.ROUT; no longer U$2.ROUT
- net N$35: now also U$6.!RSTB; no longer U$2.!RSTB
- net N$59: now also U$6.VHFI; no longer U$2.VHFI
- net N$68: now also U$6.ABYP; no longer U$2.ABYP
- net N$69: now also U$6.DACREF; no longer U$2.DACREF
- net N$70: now also U$6.DBYP; no longer U$2.DBYP
- net SCL: now also U$6.SCLK; no longer U$2.SCLK
- net SDA: now also U$6.MOSI; no longer U$2.MOSI
