File: pcb/RGBClock/Mainboard.brd (EAGLE design)
At the start: 99.8 x 70.1 mm, 102 parts, among them IC1 MCP23017SO, IC2 LT1763CS8-1.5, K1 G6K-2F, K2 G6K-2F, K3 G6K-2F, K4 G6K-2F, Q1 32.768KHz, U1 MAX6369KA+T, U10 NX3L1G384GW, U11 NX3L1G384GW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

Commit message: As send to JCLPCB
Routing:
- net N$26: track 5.50 -> 6.14 mm
Changed lines of the file:
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@@
 <setting verticaltext="up"/>
 </settings>
-<grid distance="0.5" unitdist="mm" unit="mm" style="lines" multiple="1" display="no" altdistance="0.025" altunitdist="inch" altunit="mm"/>
+<grid distance="0.05" unitdist="mm" unit="mm" style="lines" multiple="1" display="no" altdistance="0.025" altunitdist="inch" altunit="mm"/>
 <layers>
 <layer number="1" name="Top" color="4" fill="1" visible="yes" active="yes"/>
-<layer number="16" name="Bottom" color="1" fill="1" visible="yes" active="yes"/>
+<layer number="16" name="Bottom" color="1" fill="1" visible="no" active="yes"/>
 <layer number="17" name="Pads" color="2" fill="1" visible="yes" active="yes"/>
 <layer number="18" name="Vias" color="2" fill="1" visible="yes" active="yes"/>
@@
 <wire x1="21.5647" y1="44.2743" x2="21.5647" y2="43.5102" width="0.254" layer="1"/>
 <wire x1="15.8242" y1="47.625" x2="14.5033" y2="47.625" width="0.254" layer="1"/>
-<wire x1="63.3" y1="14.15" x2="63.9553" y2="14.15" width="0.254" layer="1"/>
 <wire x1="30.3128" y1="3.744" x2="31.4152" y2="2.6416" width="0.254" layer="1"/>
 <wire x1="31.4152" y1="2.6416" x2="33.5788" y2="2.6416" width="0.254" layer="1"/>
@@
 <wire x1="27.5717" y1="8.3726" x2="27.5717" y2="6.416" width="0.254" layer="1"/>
 <wire x1="28.702" y1="6.416" x2="27.5717" y2="6.416" width="0.254" layer="1"/>
-<wire x1="63.3" y1="14.9303" x2="63.398" y2="15.0283" width="0.254" layer="1"/>
-<wire x1="63.398" y1="15.0283" x2="63.398" y2="17.926" width="0.254" layer="1"/>
+<wire x1="63.398" y1="17.926" x2="63.398" y2="15.0283" width="0.254" layer="1"/>
 <wire x1="58.5741" y1="34.036" x2="58.6487" y2="34.036" width="0.254" layer="1"/>
 <wire x1="58.4994" y1="34.036" x2="58.5741" y2="34.036" width="0.254" layer="1"/>
@@
 <wire x1="2.608" y1="11.176" x2="2.608" y2="12.2315" width="0.254" layer="16"/>
 <wire x1="24.13" y1="11.67" x2="24.13" y2="10.0697" width="0.254" layer="16"/>
-<wire x1="63.9553" y1="14.15" x2="63.9553" y2="10.067" width="0.254" layer="1"/>
 <wire x1="33.5788" y1="6.9596" x2="32.6643" y2="6.9596" width="0.254" layer="1"/>
 <wire x1="29.8323" y1="6.416" x2="32.1207" y2="6.416" width="0.254" layer="1"/>
@@
 <wire x1="49.9974" y1="18.45" x2="49.9974" y2="18.95" width="0.254" layer="1"/>
 <wire x1="75.0823" y1="7.9756" x2="66.0467" y2="7.9756" width="0.254" layer="1"/>
-<wire x1="66.0467" y1="7.9756" x2="63.9553" y2="10.067" width="0.254" layer="1"/>
+<wire x1="66.0467" y1="7.9756" x2="63.96115" y2="10.06115" width="0.254" layer="1"/>
+<wire x1="63.96115" y1="10.06115" x2="63.9553" y2="10.067" width="0.254" layer="1"/>
 <wire x1="54.483" y1="59.3598" x2="54.483" y2="60.6807" width="0.254" layer="1"/>
 <wire x1="54.483" y1="60.6807" x2="54.5808" y2="60.6807" width="0.254" layer="1"/>
@@
 <wire x1="29.21" y1="44.704" x2="29.21" y2="43.6625" width="0.254" layer="16"/>
 <wire x1="63.9553" y1="10.067" x2="62.483" y2="10.067" width="0.254" layer="1"/>
-<wire x1="62.483" y1="10.067" x2="61.7" y2="10.85" width="0.254" layer="1"/>
-<wire x1="61.7" y1="10.85" x2="61.0447" y2="10.85" width="0.254" layer="1"/>
+<wire x1="62.483" y1="10.067" x2="61.65" y2="10.85" width="0.254" layer="1"/>
 <wire x1="38.1" y1="46.116" x2="37.3197" y2="46.116" width="0.254" layer="1"/>
 <wire x1="3.556" y1="27.178" x2="3.556" y2="26.1365" width="0.254" layer="16"/>
@@
 <wire x1="53.5" y1="14.3" x2="53.5" y2="13.5947" width="0.254" layer="1"/>
 <via x="30.3128" y="3.744" extent="1-16" drill="0.6096" diameter="1.016"/>
-<wire x1="63.3" y1="14.15" x2="63.3" y2="14.9303" width="0.254" layer="1"/>
 <wire x1="50.522" y1="11.9036" x2="50.522" y2="12.2833" width="0.254" layer="1"/>
 <wire x1="50.522" y1="11.303" x2="50.522" y2="11.9036" width="0.254" layer="1"/>
@@
 <via x="36" y="24" extent="1-16" drill="0.6096" diameter="1.016"/>
 <via x="43.5" y="29" extent="1-16" drill="0.6096" diameter="1.016"/>
+<wire x1="63.398" y1="15.0283" x2="63.3" y2="12.95" width="0.254" layer="1"/>
+<wire x1="63.3" y1="12.95" x2="63.3" y2="12.091975" width="0.254" layer="1"/>
+<wire x1="63.9552" y1="10.0671" x2="63.96115" y2="10.06115" width="0.254" layer="1"/>
+<wire x1="63.3" y1="12.091975" x2="63.9552" y2="11.436775" width="0.254" layer="1"/>
+<wire x1="63.9552" y1="11.436775" x2="63.9552" y2="10.0671" width="0.254" layer="1"/>
+<wire x1="61.65" y1="10.85" x2="61.0447" y2="10.85" width="0.254" layer="1"/>
 </signal>
 <signal name="N$39">
@@
 <contactref element="U$6" pad="16"/>
 <contactref element="U$2" pad="3"/>
-<wire x1="61.7" y1="14.15" x2="61.0447" y2="14.15" width="0.254" layer="1"/>
 <wire x1="57.15" y1="16.45" x2="58.7447" y2="16.45" width="0.254" layer="1"/>
-<wire x1="58.7447" y1="16.45" x2="61.0447" y2="14.15" width="0.254" layer="1"/>
+<wire x1="58.7447" y1="16.45" x2="61.65" y2="12.95" width="0.254" layer="1"/>
 </signal>
 <signal name="N$34" class="4">
@@
 <contactref element="U$6" pad="15"/>
 <contactref element="U$2" pad="1"/>
-<wire x1="62.6447" y1="10.85" x2="62.6447" y2="11.1606" width="0.254" layer="1"/>
-<wire x1="62.6447" y1="11.1606" x2="57.8553" y2="15.95" width="0.254" layer="1"/>
-<wire x1="57.15" y1="15.95" x2="57.8553" y2="15.95" width="0.254" layer="1"/>
-<wire x1="63.3" y1="10.85" x2="62.6447" y2="10.85" width="0.254" layer="1"/>
+<wire x1="61.572175" y1="12.1698" x2="62.3052" y2="11.436775" width="0.254" layer="1"/>
+<wire x1="61.572175" y1="12.1698" x2="61.188225" y2="12.1698" width="0.254" layer="1"/>
+<wire x1="61.188225" y1="12.1698" x2="59.7061" y2="13.651925" width="0.254" layer="1"/>
+<wire x1="59.7061" y1="13.651925" x2="59.7061" y2="14.0904" width="0.254" layer="1"/>
+<wire x1="59.7061" y1="14.0904" x2="57.8465" y2="15.95" width="0.254" layer="1"/>
+<wire x1="57.8465" y1="15.95" x2="57.15" y2="15.95" width="0.254" layer="1"/>
+<wire x1="62.3052" y1="11.436775" x2="63.3" y2="10.85" width="0.254" layer="1"/>
 </signal>
 </signals>

Commit message: -dab documentation -bom Mainboard.b#1 -small changes pcb
Connections:
- removed net N$62: U$6.5
- net +3V3: now also U$6.5
Routing:
- net +1.8V: track 62.8 -> 60.2 mm
Changed lines of the file:
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@@
 <wire x1="25.654" y1="3.744" x2="25.654" y2="4.7243" width="0.254" layer="1"/>
 <wire x1="20.574" y1="42.2148" x2="21.5647" y2="42.2148" width="0.254" layer="1"/>
+<contactref element="U$6" pad="5"/>
+<wire x1="52" y1="21.1" x2="53" y2="14.3" width="0" layer="19" extent="1-1"/>
 </signal>
 <signal name="+5V" class="2">
@@
 <contactref element="C11" pad="1"/>
 <contactref element="C13" pad="1"/>
-<contactref element="C28" pad="2"/>
 <contactref element="C29" pad="2"/>
 <contactref element="U$6" pad="12"/>
@@
 <wire x1="48.128" y1="26.908" x2="48.128" y2="25.8277" width="0.254" layer="16"/>
 <wire x1="37.98" y1="16.256" x2="39.4103" y2="16.256" width="0.254" layer="16"/>
-<wire x1="45.17" y1="18.304" x2="42.58" y2="18.304" width="0.254" layer="1"/>
 <wire x1="59.83" y1="11.692" x2="58.8497" y2="11.692" width="0.254" layer="16"/>
 <wire x1="58.8497" y1="11.692" x2="58.8497" y2="11.7312" width="0.254" layer="16"/>
@@
 <wire x1="36.5497" y1="17.526" x2="36.5497" y2="16.256" width="0.254" layer="16"/>
 <wire x1="48.128" y1="29.248" x2="48.128" y2="26.908" width="0.254" layer="16"/>
+<contactref element="C28" pad="2"/>
+<wire x1="45.17" y1="18.304" x2="42.58" y2="18.304" width="0" layer="19" extent="1-1"/>
 </signal>
 <signal name="N$26" class="4">
@@
 <wire x1="5.454" y1="20.2" x2="3.556" y2="22.098" width="0.762" layer="16"/>
 </signal>
-<signal name="N$62" class="4">
-<contactref element="U$6" pad="5"/>
-</signal>
 <signal name="N$2">
