File: pcb/RGBClock/Mainboard.brd (EAGLE design)
At the start: 99.8 x 70.1 mm, 102 parts, among them IC1 MCP23017SO, IC2 LT1763CS8-1.5, K1 G6K-2F, K2 G6K-2F, K3 G6K-2F, K4 G6K-2F, Q1 32.768KHz, U1 MAX6369KA+T, U10 NX3L1G384GW, U11 NX3L1G384GW, U13 DRV612PW, U14 2N7002-7-F, U15 2N7002-7-F, U16 2N7002-7-F, U17 2N7002-7-F, U2 TXS0102DCUR, U3 P82B96DR, U4 LM2675M-5.0, U5 DS1338Z-33+, U7 TPS71533DCKR, U8 NX3L1G384GW, U9 NX3L1G384GW, X2 43045-0400, X3 CON-LUMBERG_1503_09, X4 CON-LUMBERG_1503_09, X5 43045-0800, X6 ST-SMB-H

Commit message: Voor optimalisatie (v2.1)
Parts:
- removed IC2: LT1763CS8-1.5, Mainboard:LINEAR-TECHNOLOGY_SOIC8
- removed TP-5V: TESTPAD_TPSTP10SQ, Mainboard:TESTPAD_TP10SQ
- removed TP6, TP7: TESTPAD_TPTP07SQ, Mainboard:TESTPAD_TP07SQ
- removed U7: TPS71533DCKR, Mainboard:TEXAS_SOT65P210X110-5N
- removed X3, X4: CON-LUMBERG_1503_09, Mainboard:CON-LUMBERG_1503_09
- added C15, C30: 100n, Mainboard:RCL_C0805
- added C18, C31, C32, C33, C34, C35: 1u, Mainboard:RCL_C0805
- added TP1, TP8, TP9: PTR1PAD1-13, testpad:P1-13
- added U$10: TPS79133, Mainboard:SOT23-5
- added U$11, U$12: FC68131FC68131, Mainboard:FC68131
- added U$7, U$8, U$9: TPS79118, Mainboard:SOT23-5
- C14: value 0,47u -> 1u
- C4: value 10n -> 1u
- D1: value MUR480ERLG -> B340-13-F; device Mainboard:DIODE_DO41-10 -> Mainboard:DIODE_DO-214AC
- LED1: value 5mm Led -> (none); device Mainboard:LED_LED5MM -> led:CHIP-LED0805
- moved C6 30.2 mm to (64.4, 4.47), flipped to the top, turned to 270 degrees
- moved C4 29.3 mm to (61.2, 7.97), flipped to the top, turned to 0 degrees
- moved Q1 9.68 mm to (33.6, 33.1), turned to 270 degrees
- moved D1 9.64 mm to (25.6, 65.8)
- moved C14 7.24 mm to (76.7, 26.8), turned to 180 degrees
- moved LED1 5.44 mm to (25.9, 60.6), turned to 90 degrees
- moved C7 5.26 mm to (73.5, 30.4), turned to 90 degrees
- moved R12 4.37 mm to (95.9, 27.0)
- moved R13 4.26 mm to (96.1, 21.4), turned to 0 degrees
- moved C29 4.02 mm to (44.4, 23.2), flipped to the bottom
- moved C28 3.96 mm to (42.3, 23.2), flipped to the bottom
- moved R1 2.93 mm to (25.9, 57.5)
- moved U$6 2.69 mm to (51.8, 19.5)
- moved C22 2.32 mm to (59.5, 10.6)
- moved C20 2.04 mm to (87.7, 19.9), turned to 180 degrees
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Connections:
- removed net +1.8V: C11.1, C12.1, C13.1, C22.1, C28.2, C29.2, C4.1, IC2.1, IC2.2, U$6.12, U$6.35, U$6.37
- new net +1.8-MEM: C11.1, C13.1, C31.1, U$6.35, U$9.5
- new net +1.8-VA: C12.1, C22.1, C4.1, U$6.12, U$7.5
- new net +1.8-VCORE: C18.1, C28.2, C29.2, U$6.37, U$8.5
- new net N$39: C33.2, C6.1, U$7.4
- new net N$62: C30.1, C35.2, U$9.4
- new net N$65: C32.2, C7.1, U$10.4
- net +3V3: now also U$10.5; no longer U7.5
- net +5V: now also C32.1, C33.1, C34.1, C35.1, TP1.TP, U$10.1, U$7.1, U$8.1, U$9.1; no longer C6.1, C7.1, IC2.5, IC2.8, TP-5V.TP, U7.4
- net GND: now also C15.2, C18.2, C30.2, C31.2, C4.2, CON1.14, CON1.20, CON1.25, CON1.9, LED1.C, U$10.2, U$10.3, U$11.GND, U$12.GND, U$7.2, U$7.3, U$8.2, U$8.3, U$9.2, U$9.3; no longer IC2.3, IC2.6, IC2.7, LED1.K, U7.2, X3.1, X4.1
- net N$4: now also CON1.4
- net N$40: now also U$12.LEFT; no longer X4.2, X4.4
- net N$44: now also U$12.RIGHT; no longer X4.3, X4.5
- net N$47: now also U$11.LEFT; no longer X3.2, X3.4
- net N$49: now also U$11.RIGHT; no longer X3.3, X3.5
- net N$58: now also C15.1, C34.2, U$8.4; no longer C4.2, IC2.4
- net SCL: now also TP8.TP; no longer TP6.TP
- net SDA: now also TP9.TP; no longer TP7.TP
Routing:
- net +3V3: track 243.0 -> 309.6 mm, vias 1 -> 2
- net +1.8V: track 60.2 -> 0.00 mm, vias 3 -> 0
- net +1.8-MEM: track 0.00 -> 28.9 mm, vias 0 -> 2
- net +5V: track 166.7 -> 195.5 mm, vias 0 -> 2
- net SDA: track 99.5 -> 123.0 mm, vias 4 -> 1
- net GND: track 613.9 -> 635.1 mm, vias 10 -> 4
- net N$36: track 36.3 -> 15.7 mm
- net N$22: track 34.2 -> 51.0 mm, vias 1 -> 0
- net +1.8-VA: track 0.00 -> 16.3 mm, vias 0 -> 1
- net +1.8-VCORE: track 0.00 -> 15.8 mm, vias 0 -> 1
- net N$53: track 36.3 -> 24.6 mm, vias 0 -> 2
- net N$59: track 13.6 -> 23.7 mm
- net N$44: track 18.7 -> 8.93 mm
- net N$38: track 46.6 -> 37.6 mm
- net N$17: track 5.03 -> 13.8 mm
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
Commit message: Ver 2.1; as send to jclpcb
Routing:
- net N$59: track 23.7 -> 13.8 mm
- net GND: track 635.1 -> 633.9 mm, vias 4 -> 9
Other:
- board text added: "Mainboard V2.1"
Changed lines of the file:
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@@
 <hole x="3.048" y="3.302" drill="3.2"/>
 <hole x="3.048" y="67.056" drill="3.2"/>
+<text x="76.1" y="1.45" size="1.778" layer="1">Mainboard V2.1</text>
 </plain>
 <attributes>
@@
 <wire x1="33.6398" y1="5.1524" x2="34.4933" y2="4.2989" width="0.254" layer="1"/>
 <wire x1="34.4933" y1="4.2989" x2="34.4933" y2="2.6416" width="0.254" layer="1"/>
-<wire x1="50.322" y1="10.658" x2="52" y2="12.336" width="0.254" layer="1"/>
-<wire x1="52" y1="12.336" x2="52" y2="15.35" width="0.254" layer="1"/>
 <wire x1="38.8845" y1="11.67" x2="38.8845" y2="11.0175" width="0.254" layer="16"/>
 <wire x1="38.8845" y1="11.0175" x2="42.012" y2="7.89" width="0.254" layer="16"/>
@@
 <vertex x="0" y="70.1"/>
 </polygon>
+<via x="52.2" y="13.35" extent="1-16" drill="0.6096" diameter="1.016"/>
+<wire x1="51.5" y1="15.35" x2="52.159465625" y2="13.4658125" width="0.254" layer="1"/>
+<wire x1="52.159465625" y1="13.4658125" x2="52.2" y2="13.35" width="0.254" layer="1"/>
+<wire x1="53" y1="15.35" x2="52.159465625" y2="13.4658125" width="0.254" layer="1"/>
+<via x="58.8" y="21.3" extent="1-16" drill="0.6096" diameter="1.016"/>
+<via x="55.7" y="25.25" extent="1-16" drill="0.6096" diameter="1.016"/>
+<via x="45.1" y="15.3" extent="1-16" drill="0.6096" diameter="1.016"/>
+<via x="43.8" y="19.3" extent="1-16" drill="0.6096" diameter="1.016"/>
 </signal>
 <signal name="+3V3" class="4">
@@
 <wire x1="45.47" y1="10.903" x2="45.8458" y2="10.5272" width="0.254" layer="1"/>
 <wire x1="45.8458" y1="10.5272" x2="46.1976" y2="10.5272" width="0.254" layer="1"/>
-<wire x1="53.548" y1="9.9227" x2="54.0519" y2="9.4188" width="0.254" layer="1"/>
-<wire x1="54.0519" y1="9.4188" x2="54.0519" y2="7.3141" width="0.254" layer="1"/>
-<wire x1="54.0519" y1="7.3141" x2="53.2474" y2="6.5096" width="0.254" layer="1"/>
-<wire x1="53.2474" y1="6.5096" x2="47.0095" y2="6.5096" width="0.254" layer="1"/>
-<wire x1="47.0095" y1="6.5096" x2="46.1976" y2="7.3215" width="0.254" layer="1"/>
-<wire x1="46.1976" y1="7.3215" x2="46.1976" y2="10.5272" width="0.254" layer="1"/>
 <wire x1="48.822" y1="10.903" x2="47.9917" y2="10.903" width="0.254" layer="1"/>
-<wire x1="53.548" y1="10.903" x2="53.548" y2="9.9227" width="0.254" layer="1"/>
 <wire x1="53.548" y1="11.3932" x2="53.548" y2="10.903" width="0.254" layer="1"/>
 <wire x1="53.548" y1="11.3932" x2="53.548" y2="11.8833" width="0.254" layer="1"/>
-<wire x1="53.5" y1="15.35" x2="53.5" y2="11.9313" width="0.254" layer="1"/>
+<wire x1="53.5" y1="15.35" x2="53.5" y2="12.35" width="0.254" layer="1"/>
+<wire x1="53.5" y1="12.35" x2="53.5" y2="11.9313" width="0.254" layer="1"/>
 <wire x1="53.5" y1="11.9313" x2="53.548" y2="11.8833" width="0.254" layer="1"/>
+<wire x1="48.822" y1="10.903" x2="49.4" y2="12.35" width="0.254" layer="1"/>
+<wire x1="49.4" y1="12.35" x2="53.5" y2="12.35" width="0.254" layer="1"/>
 </signal>
 <signal name="N$61">

Commit message: as send to Jclpcb (ver 1.3)
Parts:
- removed C1: 100n, Mainboard:RCL_C0805
- removed C5: 594D686X0010C2T, Mainboard:MYCOMPONENTS_594D-B
- removed D4: B130-13-F, Mainboard:DIODE_DO-214AC
- removed L1: SRR1240-680M, Mainboard:BOURNS_BY_ELEMENT14_BATCH_1_SRR1240
- removed R14: A2-1, Mainboard:RESISTOR_R0402:1
- removed R15: A2-0, Mainboard:RESISTOR_R0402:1
- removed R16: A1-1, Mainboard:RESISTOR_R0402:1
- removed R17: A1-0, Mainboard:RESISTOR_R0402:1
- removed R18: A0-1, Mainboard:RESISTOR_R0402:1
- removed R19: A0-0, Mainboard:RESISTOR_R0402:1
- removed U4: LM2675M-5.0, Mainboard:TEXAS_SOIC127P620X175-8N
- added C36: 100n, Mainboard:RCL_C0805
- added IC2: R-78B5.0-2.0, linear:TO220V
- added R20: 3K48, rcl:M0805
- added SJ1: A2, jumper:SJ_2
- added SJ2: A1, jumper:SJ_2
- added SJ3: A0, jumper:SJ_2
- added U$13: SST26VF032B, Mainboard:SOIJ8
- C2: value 4,7u -> 10u
- C3: value 10n -> 10u; device Mainboard:RCL_C0805 -> Mainboard:RCL_C1206
- CON1: device Mainboard:CON-HARTING_CON26 -> con-harting:CON26
- moved C2 21.5 mm to (40.6, 66.0), turned to 0 degrees
- moved TP1 9.23 mm to (54.6, 60.1)
- moved C3 9.19 mm to (48.9, 66.0), turned to 180 degrees
- moved C28 7.23 mm to (42.0, 30.4), turned to 90 degrees
- moved C29 7.23 mm to (44.7, 30.4), turned to 90 degrees
- moved C18 6.41 mm to (41.4, 23.6)
- moved U$8 6.41 mm to (37.8, 23.6)
- moved C15 6.41 mm to (37.8, 20.4)
- moved C34 6.41 mm to (37.8, 26.7)
- moved X2 5.40 mm to (16.7, 67.4)
- moved IC1 4.45 mm to (49.0, 43.6)
- moved R6 4.31 mm to (15.9, 3.81), turned to 270 degrees
- moved CON1 3.98 mm to (4.53, 42.7)
- moved U16 3.86 mm to (59.3, 50.3)
- moved U5 3.82 mm to (38.2, 36.8)
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Connections:
- removed net N$42: IC1.16, R16.1, R17.2
- removed net N$43: IC1.17, R14.1, R15.2
- new net N$71: U$13.6, U$6.2
- new net N$72: U$13.2, U$6.47
- new net N$73: R20.2, U$13.1, U$6.1
- new net N$74: U$13.5, U$6.48
- net +3V3: now also C36.1, R20.1, SJ1.1, SJ2.1, SJ3.1, U$13.3, U$13.7, U$13.8; no longer R14.2, R16.2, R18.2
- net +5V: now also C3.1, IC2.3; no longer C5.P$1, L1.1, U4.4
- net GND: now also C3.2, C32.2, C33.2, C34.2, C35.2, C36.2, IC2.2, SJ1.3, SJ2.3, SJ3.3, U$13.4; no longer C1.2, C5.P$2, D4.A, R15.1, R17.1, R19.1, U4.6
- net N$10: now also IC1.17, SJ1.2; no longer C3.1, U4.1
- net N$11: now also IC1.16, SJ2.2; no longer C3.2, D4.C, L1.2, U4.8
- net N$39: no longer C33.2
- net N$41: now also SJ3.2; no longer R18.1, R19.2
- net N$58: no longer C34.2
- net N$62: no longer C35.2
- net N$65: no longer C32.2
- net VCC: now also IC2.1; no longer C1.1, U4.7
Routing:
- net SCL: track 93.2 -> 138.7 mm, vias 1 -> 3
- net +1.8-MEM: track 28.9 -> 68.4 mm
- net N$33: track 36.9 -> 63.6 mm
- net SDA: track 123.0 -> 103.9 mm, vias 1 -> 3
- net N$73: track 0.00 -> 19.1 mm, vias 0 -> 1
- net N$72: track 0.00 -> 16.3 mm, vias 0 -> 1
- net +5V: track 195.5 -> 181.5 mm
- net N$22: track 51.0 -> 64.6 mm
- net N$71: track 0.00 -> 13.0 mm, vias 0 -> 1
- net GND: track 633.9 -> 645.9 mm, vias 9 -> 17
- net N$37: track 17.1 -> 28.2 mm
- net N$42: track 9.92 -> 0.00 mm
- net N$74: track 0.00 -> 9.16 mm, vias 0 -> 1
- net N$11: track 17.4 -> 8.62 mm
- net VCC: track 145.5 -> 137.6 mm
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Other:
- board text added: "0-1"
- board text added: "A0"
- board text added: "A1"
- board text added: "A2"
- board text added: "Mainboard V2.2"
- board text removed: "Mainboard V2.1"

Commit message: As send to jclpcb
Parts:
- moved C26 3.05 mm to (53.8, 29.5)
- moved C27 3.05 mm to (53.8, 31.8)
- moved C12 1.83 mm to (58.0, 11.7)
- moved C22 1.83 mm to (58.0, 9.59)
- moved IC2 1.83 mm to (43.6, 63.7)
- moved U$2 1.14 mm to (63.3, 12.8), turned to 270 degrees
- moved C29 0.57 mm to (44.4, 30.9)
- moved C13 0.57 mm to (49.5, 31.0)
- moved C21 0.51 mm to (87.6, 30.7)
- moved C11 0.51 mm to (47.2, 31.0)
- moved C28 0.51 mm to (42.0, 30.9)
Connections:
- net GND: now also U$2.1, U$2.3; no longer U$2.2, U$2.4
- net N$2: now also U$2.2; no longer U$2.1
- net N$26: now also U$2.4; no longer U$2.3
Routing:
- net N$16: track 15.8 -> 84.0 mm
- net +1.8-MEM: track 68.4 -> 34.0 mm
- net +3V3: track 308.4 -> 342.1 mm, vias 7 -> 5
- net N$33: track 63.6 -> 36.6 mm
- net N$18: track 18.3 -> 34.9 mm
- net N$37: track 28.2 -> 16.8 mm
- net SDA: track 103.9 -> 95.7 mm, vias 3 -> 2
- net N$19: track 22.5 -> 30.3 mm
- net SCL: track 138.7 -> 131.5 mm, vias 3 -> 2
- net N$40: track 22.9 -> 29.6 mm
- net N$17: track 8.34 -> 14.3 mm
- net GND: track 645.9 -> 642.4 mm, vias 17 -> 10
- net N$26: track 7.99 -> 11.2 mm
- net N$70: track 24.0 -> 26.9 mm
- net N$31: track 47.7 -> 44.9 mm
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Other:
- board text added: "Mainboard V2.3"
- board text removed: "Mainboard V2.2"

Commit message: Send to jclpcb
Parts:
- added R14: 10k, rcl:M0805
- added SPI: TXS0104E, Mainboard:TEXAS_SOP65P640X120-14N
- moved IC2 0.76 mm to (43.6, 64.5)
Connections:
- new net CE0: CON1.24, SPI.5
- new net MISO: CON1.21, SPI.3
- new net MOSI: CON1.19, SPI.2
- new net SCLK: CON1.23, SPI.4
- new net SI-MISO: SPI.12, U$6.32
- new net SI_MOSI: SPI.13, U$6.31
- new net SI_SCLK: SPI.11, U$6.30
- new net SI_SSB: SPI.10, U$6.29
- net +3V3: now also SPI.14; no longer U$6.5
- net GND: now also R14.1, SPI.7, U$6.5; no longer U$6.29, U$6.32
- net N$8: now also R14.2, SPI.1, SPI.8
- net SCL: no longer U$6.30
- net SDA: no longer U$6.31
Routing:
- net N$16: track 84.0 -> 18.3 mm, vias 0 -> 1
- net SCL: track 131.5 -> 71.6 mm
- net +3V3: track 342.1 -> 295.8 mm
- net CE0: track 0.00 -> 37.5 mm
- net GND: track 642.4 -> 606.3 mm, vias 10 -> 18
- net SCLK: track 0.00 -> 33.8 mm
- net MISO: track 0.00 -> 32.0 mm
- net SI_SSB: track 0.00 -> 30.9 mm, vias 0 -> 1
- net SI_SCLK: track 0.00 -> 30.1 mm, vias 0 -> 1
- net MOSI: track 0.00 -> 30.1 mm
- net N$8: track 16.5 -> 46.5 mm
- net SI_MOSI: track 0.00 -> 29.6 mm, vias 0 -> 1
- net SI-MISO: track 0.00 -> 28.2 mm, vias 0 -> 1
- net N$36: track 16.1 -> 41.9 mm
- net SDA: track 95.7 -> 75.7 mm, vias 2 -> 1
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Other:
- board text added: "Mainboard V2.4"
- board text removed: "Mainboard V2.3"

Commit message: - some comments
Connections:
- net N$71 renamed NVSCLK
- net N$72 renamed NVMISO
- net N$73 renamed NVSSB
- net N$74 renamed NVMOSI
Changed lines of the file:
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@@
 <wire x1="47.244" y1="31.938" x2="48.3243" y2="31.938" width="0.254" layer="16"/>
 </signal>
-<signal name="N$71">
+<signal name="NVSCLK">
 <contactref element="U$13" pad="6"/>
 <contactref element="U$6" pad="2"/>
@@
 <via x="42.3764" y="14.6567" extent="1-16" drill="0.6096" diameter="1.016"/>
 </signal>
-<signal name="N$73">
+<signal name="NVSSB">
 <contactref element="U$13" pad="1"/>
 <contactref element="U$6" pad="1"/>
@@
 <wire x1="34.55" y1="12.8" x2="34.55" y2="13.9303" width="0.254" layer="16"/>
 </signal>
-<signal name="N$74">
+<signal name="NVMOSI">
 <contactref element="U$13" pad="5"/>
 <contactref element="U$6" pad="48"/>
@@
 <wire x1="40.0653" y1="18.1533" x2="41.2296" y2="16.989" width="0.254" layer="16"/>
 </signal>
-<signal name="N$72">
+<signal name="NVMISO">
 <contactref element="U$13" pad="2"/>
 <contactref element="U$6" pad="47"/>
